File: Placa de configuração LoRa/Placa de configuração LoRa.kicad_pcb (KiCad board)
At the start: 2 copper layers, 8 parts

Commit message: Add
Parts:
- removed the REF** at (152.3, 100.3)
- added REF**: R_Axial_DIN0207_L6.3mm_D2.5mm_P10.16mm_Horizontal, Resistor_THT:R_Axial_DIN0207_L6.3mm_D2.5mm_P10.16mm_Horizontal, F.Cu at (146.4, 100.3)
- moved REF** 5.70 mm to (142.5, 129.6)
- moved REF** 5.70 mm to (140.6, 87.4)
- moved REF** 5.70 mm to (143.2, 87.4)
- moved REF** 5.70 mm to (145.8, 87.4)
- moved REF** 5.70 mm to (135.5, 94.7)
- moved REF** 5.70 mm to (153.6, 89.6)
Routing:
- net Net-(A1-Pad6): track 11.1 -> 16.8 mm
- net Net-(A1-Pad29): track 50.0 -> 55.7 mm
- net +3V3: track 72.2 -> 77.9 mm
- net Net-(A1-Pad8): track 26.8 -> 32.5 mm
- net +5V: track 43.5 -> 49.2 mm
- net Net-(A1-Pad9): track 30.9 -> 36.6 mm
- net Net-(A1-Pad5): track 6.97 -> 12.0 mm
- net Net-(A1-Pad7): track 13.6 -> 17.9 mm
